File: uGetto/nano_getto/nano_getto.kicad_pcb (KiCad board)
At the start: 2 copper layers, 9 parts, among them J1 Conn_01x06_Male, SW1 SW_Push, U1 ATtiny13A-SS

Commit message: Changed attiny13a footprint to SOIC8W
Parts:
- U1: value ATtiny13A-SS -> ATtiny13A-S; footprint Package_SO:SOIC-8_3.9x4.9mm_P1.27mm -> Package_SO:SOIC-8W_5.3x5.3mm_P1.27mm
- moved U1 0.25 mm to (121.4, 116.3)
Routing:
- net Net-(SW1-Pad1): track 48.4 -> 47.0 mm
- net Net-(R1-Pad1): track 28.5 -> 27.1 mm
- net Net-(J1-Pad5): track 9.87 -> 8.45 mm
- net Net-(D1-Pad1): track 27.2 -> 25.8 mm
- net Net-(J1-Pad2): track 38.7 -> 39.8 mm
- net Net-(J1-Pad3): track 44.4 -> 43.5 mm
